File: uvmeter.brd (EAGLE design)
At the start: 100 x 80 mm, 18 parts, among them U1 ATTINY2313A, U2 ML8511-UV-SENSORSMD

Commit message: added attiny84
attiny2313 doesn’t have an onboard adc, swapping it out for an attyin84
Parts:
- added U$1: ATTINY84, SparkFun-DigitalIC:SO14
Connections:
- net N$1 renamed D10
- net N$10 renamed D12
- net N$11 renamed D11
- net N$9 renamed D13
Changed lines of the file:
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@@
 <element name="R4" library="SparkFun-Resistors" package="0805" value="" x="17.8562" y="34.417" rot="R180"/>
 <element name="R5" library="SparkFun-Resistors" package="0805" value="" x="45.72" y="7.62"/>
+<element name="U$1" library="SparkFun-DigitalIC" package="SO14" value="ATTINY84" x="4.5466" y="-5.5626">
+<attribute name="PROD_ID" value="IC-11285" x="4.5466" y="-5.5626" size="1.778" layer="27" display="off"/>
+</element>
 </elements>
 <signals>
@@
 <wire x1="17.78" y1="30.48" x2="18.7562" y2="34.417" width="0" layer="19" extent="1-1"/>
 </signal>
-<signal name="N$9">
+<signal name="D13">
 <contactref element="U1" pad="16"/>
 </signal>
-<signal name="N$10">
+<signal name="D12">
 <contactref element="U1" pad="15"/>
 </signal>
-<signal name="N$11">
+<signal name="D11">
 <contactref element="U1" pad="14"/>
 </signal>
@@
 <contactref element="U2" pad="4"/>
 </signal>
-<signal name="N$1">
+<signal name="D10">
 <contactref element="U1" pad="13"/>
 </signal>
